Commit message: se arreglaron algunos errores de colisiones

File: phantom_ws/src/phantomx_pincher/phantomx_pincher_description/urdf/phantomx_pincher.urdf.xacro (robot description, xacro)
@@ -65,5 +65,5 @@
         rpy = "roll pitch yaw"
     -->
-    <origin xyz="0 0 0" rpy="0 0 0"/>
+    <origin xyz="0.01325 0 0.016" rpy="0 0 0"/>
   </joint>
   <!-- Arm -->

File: phantom_ws/src/phantomx_pincher/phantomx_pincher_moveit_config/srdf/phantomx_pincher.xacro (robot description, xacro)
@@ -96,8 +96,10 @@
     <disable_collisions link1="${prefix}arm_elbow_F10_0_link" link2="${prefix}gripper_servo_link"
       reason="Never" />
+    <!--
     <disable_collisions link1="${prefix}arm_elbow_F10_0_link" link2="${prefix}task_board_link"
       reason="Never" />
     <disable_collisions link1="${prefix}arm_elbow_F10_0_link" link2="${prefix}task_board_mount_link"
       reason="Never" />
+    -->
     <disable_collisions link1="${prefix}arm_elbow_F10_1_link" link2="${prefix}arm_elbow_F10_2_link"
       reason="Adjacent" />
@@ -136,8 +138,10 @@
     <disable_collisions link1="${prefix}arm_elbow_F10_1_link" link2="${prefix}gripper_servo_link"
       reason="Never" />
+    <!--
     <disable_collisions link1="${prefix}arm_elbow_F10_1_link" link2="${prefix}task_board_link"
       reason="Never" />
     <disable_collisions link1="${prefix}arm_elbow_F10_1_link" link2="${prefix}task_board_mount_link"
       reason="Never" />
+    -->
     <disable_collisions link1="${prefix}arm_elbow_F10_2_link" link2="${prefix}arm_elbow_F3_0_link"
       reason="Adjacent" />
@@ -174,8 +178,10 @@
     <disable_collisions link1="${prefix}arm_elbow_F10_2_link" link2="${prefix}gripper_servo_link"
       reason="Never" />
+    <!--
     <disable_collisions link1="${prefix}arm_elbow_F10_2_link" link2="${prefix}task_board_link"
       reason="Never" />
     <disable_collisions link1="${prefix}arm_elbow_F10_2_link" link2="${prefix}task_board_mount_link"
       reason="Never" />
+    -->
     <disable_collisions link1="${prefix}arm_elbow_F3_0_link" link2="${prefix}arm_elbow_flex_link"
       reason="Never" />
@@ -240,8 +246,10 @@
     <disable_collisions link1="${prefix}arm_elbow_flex_link" link2="${prefix}gripper_servo_link"
       reason="Never" />
+    <!--
     <disable_collisions link1="${prefix}arm_elbow_flex_link" link2="${prefix}task_board_link"
       reason="Never" />
     <disable_collisions link1="${prefix}arm_elbow_flex_link" link2="${prefix}task_board_mount_link"
       reason="Never" />
+    -->
     <disable_collisions link1="${prefix}arm_elbow_flex_servo_link"
       link2="${prefix}arm_shoulder_F10_0_link" reason="Never" />
@@ -266,6 +274,8 @@
     <disable_collisions link1="${prefix}arm_elbow_flex_servo_link"
       link2="${prefix}arm_wrist_flex_servo_link" reason="Never" />
+    <!--
     <disable_collisions link1="${prefix}arm_elbow_flex_servo_link" link2="${prefix}base_mount_link"
       reason="Never" />
+      -->
     <disable_collisions link1="${prefix}arm_elbow_flex_servo_link"
       link2="${prefix}gripper_finger1_link" reason="Never" />
@@ -276,8 +286,10 @@
     <disable_collisions link1="${prefix}arm_elbow_flex_servo_link"
       link2="${prefix}gripper_servo_link" reason="Never" />
+    <!--
     <disable_collisions link1="${prefix}arm_elbow_flex_servo_link" link2="${prefix}task_board_link"
       reason="Never" />
     <disable_collisions link1="${prefix}arm_elbow_flex_servo_link"
       link2="${prefix}task_board_mount_link" reason="Never" />
+      -->
     <disable_collisions link1="${prefix}arm_shoulder_F10_0_link"
       link2="${prefix}arm_shoulder_F10_1_link" reason="Adjacent" />
@@ -300,6 +312,8 @@
     <disable_collisions link1="${prefix}arm_shoulder_F10_0_link"
       link2="${prefix}arm_wrist_flex_servo_link" reason="Never" />
+    <!--
     <disable_collisions link1="${prefix}arm_shoulder_F10_0_link" link2="${prefix}base_mount_link"
       reason="Never" />
+    -->
     <disable_collisions link1="${prefix}arm_shoulder_F10_0_link"
       link2="${prefix}gripper_finger1_link" reason="Never" />
@@ -310,8 +324,10 @@
     <disable_collisions link1="${prefix}arm_shoulder_F10_0_link" link2="${prefix}gripper_servo_link"
       reason="Never" />
+    <!--
     <disable_collisions link1="${prefix}arm_shoulder_F10_0_link" link2="${prefix}task_board_link"
       reason="Never" />
     <disable_collisions link1="${prefix}arm_shoulder_F10_0_link"
       link2="${prefix}task_board_mount_link" reason="Never" />
+    -->
     <disable_collisions link1="${prefix}arm_shoulder_F10_1_link"
       link2="${prefix}arm_shoulder_F10_2_link" reason="Adjacent" />
@@ -332,6 +348,8 @@
     <disable_collisions link1="${prefix}arm_shoulder_F10_1_link"
       link2="${prefix}arm_wrist_flex_servo_link" reason="Never" />
+    <!--
     <disable_collisions link1="${prefix}arm_shoulder_F10_1_link" link2="${prefix}base_mount_link"
       reason="Never" />
+    -->
     <disable_collisions link1="${prefix}arm_shoulder_F10_1_link"
       link2="${prefix}gripper_finger1_link" reason="Never" />
@@ -342,8 +360,10 @@
     <disable_collisions link1="${prefix}arm_shoulder_F10_1_link" link2="${prefix}gripper_servo_link"
       reason="Never" />
+    <!--
     <disable_collisions link1="${prefix}arm_shoulder_F10_1_link" link2="${prefix}task_board_link"
       reason="Never" />
     <disable_collisions link1="${prefix}arm_shoulder_F10_1_link"
       link2="${prefix}task_board_mount_link" reason="Never" />
+    -->
     <disable_collisions link1="${prefix}arm_shoulder_F10_2_link"
       link2="${prefix}arm_shoulder_F3_0_link" reason="Adjacent" />
@@ -362,6 +382,8 @@
     <disable_collisions link1="${prefix}arm_shoulder_F10_2_link"
       link2="${prefix}arm_wrist_flex_servo_link" reason="Never" />
+    <!--
     <disable_collisions link1="${prefix}arm_shoulder_F10_2_link" link2="${prefix}base_mount_link"
       reason="Never" />
+    -->
     <disable_collisions link1="${prefix}arm_shoulder_F10_2_link"
       link2="${prefix}gripper_finger1_link" reason="Never" />
@@ -372,8 +394,10 @@
     <disable_collisions link1="${prefix}arm_shoulder_F10_2_link" link2="${prefix}gripper_servo_link"
       reason="Never" />
+    <!--
     <disable_collisions link1="${prefix}arm_shoulder_F10_2_link" link2="${prefix}task_board_link"
       reason="Never" />
     <disable_collisions link1="${prefix}arm_shoulder_F10_2_link"
       link2="${prefix}task_board_mount_link" reason="Never" />
+    -->
     <disable_collisions link1="${prefix}arm_shoulder_F3_0_link"
       link2="${prefix}arm_shoulder_lift_link" reason="Never" />
@@ -390,6 +414,8 @@
     <disable_collisions link1="${prefix}arm_shoulder_F3_0_link"
       link2="${prefix}arm_wrist_flex_servo_link" reason="Never" />
+    <!--
     <disable_collisions link1="${prefix}arm_shoulder_F3_0_link" link2="${prefix}base_mount_link"
       reason="Never" />
+    -->
     <disable_collisions link1="${prefix}arm_shoulder_F3_0_link"
       link2="${prefix}gripper_finger1_link" reason="Never" />
@@ -400,8 +426,10 @@
     <disable_collisions link1="${prefix}arm_shoulder_F3_0_link" link2="${prefix}gripper_servo_link"
       reason="Never" />
+    <!--
     <disable_collisions link1="${prefix}arm_shoulder_F3_0_link" link2="${prefix}task_board_link"
       reason="Never" />
     <disable_collisions link1="${prefix}arm_shoulder_F3_0_link"
       link2="${prefix}task_board_mount_link" reason="Never" />
+    -->
     <disable_collisions link1="${prefix}arm_shoulder_lift_link"
       link2="${prefix}arm_shoulder_lift_servo_link" reason="Adjacent" />
@@ -416,10 +444,14 @@
     <disable_collisions link1="${prefix}arm_shoulder_lift_link"
       link2="${prefix}arm_wrist_flex_servo_link" reason="Never" />
+    <!--
     <disable_collisions link1="${prefix}arm_shoulder_lift_link" link2="${prefix}base_mount_link"
       reason="Never" />
+    -->
+    <!--
     <disable_collisions link1="${prefix}arm_shoulder_lift_link" link2="${prefix}task_board_link"
       reason="Never" />
     <disable_collisions link1="${prefix}arm_shoulder_lift_link"
       link2="${prefix}task_board_mount_link" reason="Never" />
+    -->
     <disable_collisions link1="${prefix}arm_shoulder_lift_servo_link"
       link2="${prefix}arm_shoulder_pan_link" reason="Adjacent" />
@@ -430,10 +462,14 @@
     <disable_collisions link1="${prefix}arm_shoulder_lift_servo_link"
       link2="${prefix}arm_wrist_flex_servo_link" reason="Never" />
+    <!--
     <disable_collisions link1="${prefix}arm_shoulder_lift_servo_link"
       link2="${prefix}base_mount_link" reason="Never" />
+    -->
+    <!--
     <disable_collisions link1="${prefix}arm_shoulder_lift_servo_link"
       link2="${prefix}task_board_link" reason="Never" />
     <disable_collisions link1="${prefix}arm_shoulder_lift_servo_link"
       link2="${prefix}task_board_mount_link" reason="Never" />
+    -->
     <disable_collisions link1="${prefix}arm_shoulder_pan_link"
       link2="${prefix}arm_shoulder_pan_servo_link" reason="Adjacent" />
@@ -442,6 +478,9 @@
     <disable_collisions link1="${prefix}arm_shoulder_pan_link"
       link2="${prefix}arm_wrist_flex_servo_link" reason="Never" />
+    <!--
     <disable_collisions link1="${prefix}arm_shoulder_pan_link" link2="${prefix}base_mount_link"
       reason="Never" />
+    -->
+    <!--
     <disable_collisions link1="${prefix}arm_shoulder_pan_link" link2="${prefix}task_board_link"
       reason="Never" />
@@ -454,4 +493,5 @@
     <disable_collisions link1="${prefix}arm_shoulder_pan_servo_link"
       link2="${prefix}task_board_mount_link" reason="Never" />
+    -->
     <disable_collisions link1="${prefix}arm_wrist_F3_0_link" link2="${prefix}arm_wrist_flex_link"
       reason="Adjacent" />
@@ -484,8 +524,10 @@
     <disable_collisions link1="${prefix}arm_wrist_flex_servo_link"
       link2="${prefix}gripper_servo_link" reason="Never" />
+    <!--
     <disable_collisions link1="${prefix}base_mount_link" link2="${prefix}task_board_link"
       reason="Never" />
     <disable_collisions link1="${prefix}base_mount_link" link2="${prefix}task_board_mount_link"
       reason="Adjacent" />
+    -->
     <disable_collisions link1="${prefix}gripper_finger1_link" link2="${prefix}gripper_finger2_link"
       reason="Never" />
@@ -500,6 +542,8 @@
     <disable_collisions link1="${prefix}gripper_finger_base_link"
       link2="${prefix}gripper_servo_link" reason="Adjacent" />
+    <!--
     <disable_collisions link1="${prefix}task_board_link" link2="${prefix}task_board_mount_link"
       reason="Adjacent" />
+    -->
   </xacro:macro>
 </robot>
